File: Shift.sch (KiCad schematic (older format))
At the start: 3 parts

Commit message: no message
Parts:
- removed U? (x3): SN74ACT245, symbol bambouLab:SN74ACT245
Changed lines of the file:
@@
 Comment4 ""
 $EndDescr
-$Comp
-L bambouLab:SN74ACT245 U?
-U 1 1 5D990840
-P 3300 3750
-F 0 "U?" H 3275 4315 50  0000 C CNN
-F 1 "SN74ACT245" H 3275 4224 50  0000 C CNN
-F 2 "" H 3300 3750 50  0001 C CNN
-F 3 "" H 3300 3750 50  0001 C CNN
-	1    3300 3750
-	1    0    0    -1
-$EndComp
-$Comp
-L bambouLab:SN74ACT245 U?
-U 1 1 5D993E8C
-P 5500 3750
-F 0 "U?" H 5475 4315 50  0000 C CNN
-F 1 "SN74ACT245" H 5475 4224 50  0000 C CNN
-F 2 "" H 5500 3750 50  0001 C CNN
-F 3 "" H 5500 3750 50  0001 C CNN
-	1    5500 3750
-	1    0    0    -1
-$EndComp
-$Comp
-L bambouLab:SN74ACT245 U?
-U 1 1 5D994EE2
-P 7700 3750
-F 0 "U?" H 7675 4315 50  0000 C CNN
-F 1 "SN74ACT245" H 7675 4224 50  0000 C CNN
-F 2 "" H 7700 3750 50  0001 C CNN
-F 3 "" H 7700 3750 50  0001 C CNN
-	1    7700 3750
-	1    0    0    -1
-$EndComp
 $EndSCHEMATC
